File: ErgoDoxTW.kicad_pcb (KiCad board)
At the start: 2 copper layers, 182.8 x 158.9 mm, 63 parts, among them J1 3.5mm, J2 USB_C, SW0:10 SW0:3, SW0:11 SW0:2, SW0:12 SW0:1, SW0:7 SW0:6, SW0:8 SW0:5, SW0:9 SW0:4, SW1:10 SW1:3, SW1:11 SW1:2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

Commit message: v1.4 formal release
update TRRS position and silksprint
Parts:
- moved J1 0.50 mm to (86.8, 30.9)
Routing:
- net GND: track 203.7 -> 202.5 mm
- net VCC: track 149.6 -> 150.1 mm
